Commit message: Update cartesian_irrigator.urdf.xacro

File: cartesian_irrigator.urdf.xacro (robot description, xacro)
@@ -58,4 +58,7 @@
         <box size="0.18 0.18 0.18"/>
       </geometry>
+	     	<material name="Yellow2">
+				<color rgba="0.8 0.8 0 1.0"/>
+			</material>
     </visual>
   </link>
